Commit message: update mir_robot: add kinect v2 and fix pid bug

File: mir_robot/mir_description/urdf/mir.urdf.xacro (robot description, xacro)
@@ -9,4 +9,6 @@
   <!-- RG2 Gripper base -->
   <xacro:include filename="$(find robotiq_description)/urdf/robotiq_85_gripper.urdf.xacro" />
+  <!-- Kinect V2 base -->
+  <xacro:include filename="$(find kinect_v2)/urdf/kinect_v2.urdf.xacro" />
   <xacro:arg name="tf_prefix" default="" />
   <xacro:property name="tf_prefix_" value="$(arg tf_prefix)" />
@@ -18,5 +20,5 @@
   </xacro:unless>
   <xacro:mir_100 prefix="${prefix}"/>
-  <!-- MIR + UR5E + Robotiq-->
+  <!-- MIR + UR5E + Robotiq + Kinect V2-->
   <xacro:ur5e_robot prefix="${tf_prefix}_ur5e" />
   <joint name="${tf_prefix}_ur5e_fixed_joint" type="fixed">
@@ -57,5 +59,9 @@
     <child link="$(arg tf_prefix)robotiq_coupler"/>
   </joint>
-  <!-- Gazebo FT sensor plugin -->
+  <xacro:kinect_v2  parent="$(arg tf_prefix)_ur5etool0">
+    <origin xyz="0.0 0.0 0"
+            rpy="0 0 0" />
+  </xacro:kinect_v2>
+  <!-- Gazebo plugin -->
   <gazebo reference="$(arg tf_prefix)_ur5ewrist_3_joint">
     <provideFeedback>true</provideFeedback>
@@ -69,5 +75,4 @@
       </plugin>
   </gazebo>
-  <!-- Gazebo plugin -->
   <gazebo>
       <gripper name="gazebo_gripper">

Commit message: update mir robot

File: mir_robot/mir_description/urdf/mir.urdf.xacro (robot description, xacro)
@@ -8,5 +8,5 @@
   <xacro:include filename="$(find ur_description)/urdf/inc/ur5e_macro.xacro"/>
   <!-- RG2 Gripper base -->
-  <xacro:include filename="$(find robotiq_description)/urdf/robotiq_85_gripper.urdf.xacro" />
+  <!-- <xacro:include filename="$(find robotiq_description)/urdf/robotiq_85_gripper.urdf.xacro" /> -->
   <!-- Kinect V2 base -->
   <xacro:include filename="$(find kinect_v2)/urdf/kinect_v2.urdf.xacro" />
@@ -27,39 +27,6 @@
     <child link="${tf_prefix}_ur5ebase_link"/>
   </joint>
-  <link name="${tf_prefix}robotiq_coupler">
-    <visual>
-    <geometry>
-        <mesh filename="package://robotiq_description/meshes/robotiq_85_coupler.stl" />
-    </geometry>
-    <material name="flat_black"/>
-    </visual>
-    <collision>
-    <geometry>
-        <mesh filename="package://robotiq_description/meshes/robotiq_85_coupler.stl" />
-    </geometry>
-    </collision>
-    <inertial>
-    <origin xyz="2.073e-05   1.45286e-03  -1.1049e-03" rpy="0 0 0" />
-    <mass value="0.168" />
-    <inertia ixx="6.69695624e-05" ixy="5.21511788e-09" ixz="-2.74383009e-08"
-            iyy="7.85088161e-05" iyz="5.41105193e-07" izz="1.41819717e-04"/>
-    </inertial>
-  </link>
-  <xacro:robotiq_85_gripper prefix="${tf_prefix}" parent="${tf_prefix}robotiq_coupler" >
-    <origin xyz="0 0 0.004" rpy="0 ${-pi/2} ${pi}"/>
-  </xacro:robotiq_85_gripper>
-  <gazebo reference="$(arg tf_prefix)robotiq_coupler">
-    <mu1>0.9</mu1>
-    <mu2>0.9</mu2>
-    <material>Gazebo/FlatBlack</material>
-  </gazebo>
-  <joint name="$(arg tf_prefix)robotiq_coupler_joint" type="fixed">
-    <origin xyz="0 0 0.004" rpy="0 0 ${-pi/2.0}" />
-    <parent link="${tf_prefix}_ur5etool0"/>
-    <child link="$(arg tf_prefix)robotiq_coupler"/>
-  </joint>
-  <xacro:kinect_v2  parent="$(arg tf_prefix)_ur5etool0">
-    <origin xyz="0.0 0.0 0"
-            rpy="0 0 0" />
+  <xacro:kinect_v2  parent="$(arg tf_prefix)_ur5etool0" prefix="$(arg tf_prefix)">
+    <origin xyz="0.0 0.0 0" rpy="0 0 0" />
   </xacro:kinect_v2>
   <!-- Gazebo plugin -->
@@ -75,16 +42,4 @@
       </plugin>
   </gazebo>
-  <gazebo>
-      <gripper name="gazebo_gripper">
-      <grasp_check>
-          <attach_steps>2</attach_steps>
-          <detach_steps>2</detach_steps>
-          <min_contact_count>3</min_contact_count>
-      </grasp_check>
-      <gripper_link>$(arg tf_prefix)robotiq_85_left_finger_tip_link</gripper_link>
-      <gripper_link>$(arg tf_prefix)robotiq_85_right_finger_tip_link</gripper_link>
-      <palm_link>$(arg tf_prefix)robotiq_85_base_link</palm_link>
-      </gripper>
-  </gazebo>
   <xacro:controller_plugin_gazebo robot_namespace=""/>
 </robot>

Commit message: update mir robot

File: mir_robot/mir_description/urdf/mir.urdf.xacro (robot description, xacro)
@@ -27,8 +27,70 @@
     <child link="${tf_prefix}_ur5ebase_link"/>
   </joint>
-  <xacro:kinect_v2  parent="$(arg tf_prefix)_ur5etool0" prefix="$(arg tf_prefix)">
+  <!-- <xacro:kinect_v2  parent="$(arg tf_prefix)_ur5etool0" prefix="$(arg tf_prefix)">
     <origin xyz="0.0 0.0 0" rpy="0 0 0" />
-  </xacro:kinect_v2>
+  </xacro:kinect_v2> -->
+  <joint name="${tf_prefix}_camera_joint" type="fixed">
+    <axis xyz="0 1 0" />
+    <origin xyz="0 -0.06 -0.02" rpy="0 0 0"/>
+    <parent link="$(arg tf_prefix)_ur5etool0"/>
+    <child link="${tf_prefix}_camera_link"/>
+  </joint>
+  <link name="${tf_prefix}_camera_link">
+    <collision>
+      <origin xyz="0 0 0" rpy="0 0 0"/>
+      <geometry>
+    <box size="0.025 0.025 0.025"/>
+      </geometry>
+    </collision>
+    <visual>
+      <origin xyz="0 0 0" rpy="0 0 0"/>
+      <geometry>
+    <box size="0.025 0.025 0.025"/>
+      </geometry>
+      <material name="red"/>
+    </visual>
+    <inertial>
+      <mass value="1e-5" />
+      <origin xyz="0 0 0" rpy="0 0 0"/>
+      <inertia ixx="1e-6" ixy="0" ixz="0" iyy="1e-6" iyz="0" izz="1e-6" />
+    </inertial>
+  </link>
   <!-- Gazebo plugin -->
+  <!-- <gazebo reference="${tf_prefix}_camera_link">
+    <sensor type="camera" name="${tf_prefix}_camera">
+      <update_rate>30.0</update_rate>
+      <camera name="head">
+        <horizontal_fov>1.3962634</horizontal_fov>
+        <image>
+          <width>800</width>
+          <height>800</height>
+          <format>R8G8B8</format>
+        </image>
+        <clip>
+          <near>0.02</near>
+          <far>300</far>
+        </clip>
+        <noise>
+          <type>gaussian</type>
+          <mean>0.0</mean>
+          <stddev>0.007</stddev>
+        </noise>
+      </camera>
+      <plugin name="camera_controller" filename="libgazebo_ros_camera.so">
+        <alwaysOn>true</alwaysOn>
+        <updateRate>0.0</updateRate>
+        <cameraName>${tf_prefix}_camera</cameraName>
+        <imageTopicName>${tf_prefix}_camera/image_raw</imageTopicName>
+        <cameraInfoTopicName>${tf_prefix}_camera/camera_info</cameraInfoTopicName>
+        <frameName>${tf_prefix}_camera_link</frameName>
+        <hackBaseline>0.07</hackBaseline>
+        <distortionK1>0.0</distortionK1>
+        <distortionK2>0.0</distortionK2>
+        <distortionK3>0.0</distortionK3>
+        <distortionT1>0.0</distortionT1>
+        <distortionT2>0.0</distortionT2>
+      </plugin>
+    </sensor>
+  </gazebo> -->
   <gazebo reference="$(arg tf_prefix)_ur5ewrist_3_joint">
     <provideFeedback>true</provideFeedback>

Commit message: update mir robot

File: mir_robot/mir_description/urdf/mir.urdf.xacro (robot description, xacro)
@@ -7,8 +7,4 @@
   <!-- UR5E base -->
   <xacro:include filename="$(find ur_description)/urdf/inc/ur5e_macro.xacro"/>
-  <!-- RG2 Gripper base -->
-  <!-- <xacro:include filename="$(find robotiq_description)/urdf/robotiq_85_gripper.urdf.xacro" /> -->
-  <!-- Kinect V2 base -->
-  <xacro:include filename="$(find kinect_v2)/urdf/kinect_v2.urdf.xacro" />
   <xacro:arg name="tf_prefix" default="" />
   <xacro:property name="tf_prefix_" value="$(arg tf_prefix)" />
@@ -20,4 +16,5 @@
   </xacro:unless>
   <xacro:mir_100 prefix="${prefix}"/>
+  <xacro:controller_plugin_gazebo robot_namespace=""/>
   <!-- MIR + UR5E + Robotiq + Kinect V2-->
   <xacro:ur5e_robot prefix="${tf_prefix}_ur5e" />
@@ -27,18 +24,15 @@
     <child link="${tf_prefix}_ur5ebase_link"/>
   </joint>
-  <!-- <xacro:kinect_v2  parent="$(arg tf_prefix)_ur5etool0" prefix="$(arg tf_prefix)">
-    <origin xyz="0.0 0.0 0" rpy="0 0 0" />
-  </xacro:kinect_v2> -->
-  <joint name="${tf_prefix}_camera_joint" type="fixed">
+  <joint name="${tf_prefix}_camera_joint1" type="fixed">
     <axis xyz="0 1 0" />
-    <origin xyz="0 -0.06 -0.02" rpy="0 0 0"/>
-    <parent link="$(arg tf_prefix)_ur5etool0"/>
-    <child link="${tf_prefix}_camera_link"/>
+    <origin xyz="0.5 0.0 0.2" rpy="0.0 -1.5707963 0.0"/>
+    <parent link="$(arg tf_prefix)/base_link"/>
+    <child link="${tf_prefix}_camera_link1"/>
   </joint>
-  <link name="${tf_prefix}_camera_link">
+  <link name="${tf_prefix}_camera_link1">
     <collision>
       <origin xyz="0 0 0" rpy="0 0 0"/>
       <geometry>
-    <box size="0.025 0.025 0.025"/>
+        <box size="0.025 0.025 0.025"/>
       </geometry>
     </collision>
@@ -46,7 +40,6 @@
       <origin xyz="0 0 0" rpy="0 0 0"/>
       <geometry>
-    <box size="0.025 0.025 0.025"/>
+        <box size="0.025 0.025 0.025"/>
       </geometry>
-      <material name="red"/>
     </visual>
     <inertial>
@@ -57,8 +50,8 @@
   </link>
   <!-- Gazebo plugin -->
-  <!-- <gazebo reference="${tf_prefix}_camera_link">
-    <sensor type="camera" name="${tf_prefix}_camera">
-      <update_rate>30.0</update_rate>
-      <camera name="head">
+  <gazebo reference="${tf_prefix}_camera_link1">
+    <sensor type="camera" name="camera1">
+      <update_rate>100.0</update_rate>
+      <camera name="camera1">
         <horizontal_fov>1.3962634</horizontal_fov>
         <image>
@@ -79,9 +72,9 @@
       <plugin name="camera_controller" filename="libgazebo_ros_camera.so">
         <alwaysOn>true</alwaysOn>
-        <updateRate>0.0</updateRate>
-        <cameraName>${tf_prefix}_camera</cameraName>
-        <imageTopicName>${tf_prefix}_camera/image_raw</imageTopicName>
-        <cameraInfoTopicName>${tf_prefix}_camera/camera_info</cameraInfoTopicName>
-        <frameName>${tf_prefix}_camera_link</frameName>
+        <updateRate>100.0</updateRate>
+        <cameraName>camera1</cameraName>
+        <imageTopicName>image_raw_camera1</imageTopicName>
+        <cameraInfoTopicName>camera_info1</cameraInfoTopicName>
+        <frameName>${tf_prefix}_camera_link1</frameName>
         <hackBaseline>0.07</hackBaseline>
         <distortionK1>0.0</distortionK1>
@@ -92,16 +85,66 @@
       </plugin>
     </sensor>
-  </gazebo> -->
-  <gazebo reference="$(arg tf_prefix)_ur5ewrist_3_joint">
-    <provideFeedback>true</provideFeedback>
   </gazebo>
-  <gazebo>
-      <plugin name="ft_sensor_plugin" filename="libgazebo_ros_ft_sensor.so">
-      <updateRate>250.0</updateRate>
-      <topicName>wrench</topicName>
-      <gaussianNoise>0.0</gaussianNoise>
-      <jointName>$(arg tf_prefix)_ur5ewrist_3_joint</jointName>
+  <joint name="${tf_prefix}_camera_joint2" type="fixed">
+    <axis xyz="0 1 0" />
+    <origin xyz="0.0 -0.055 -0.055" rpy="0.0 -1.5707963 0.0"/>
+    <parent link="$(arg tf_prefix)_ur5etool0"/>
+    <child link="${tf_prefix}_camera_link2"/>
+  </joint>
+  <link name="${tf_prefix}_camera_link2">
+    <collision>
+      <origin xyz="0 0 0" rpy="0 0 0"/>
+      <geometry>
+        <box size="0.025 0.025 0.025"/>
+      </geometry>
+    </collision>
+    <visual>
+      <origin xyz="0 0 0" rpy="0 0 0"/>
+      <geometry>
+        <box size="0.025 0.025 0.025"/>
+      </geometry>
+    </visual>
+    <inertial>
+      <mass value="1e-5" />
+      <origin xyz="0 0 0" rpy="0 0 0"/>
+      <inertia ixx="1e-6" ixy="0" ixz="0" iyy="1e-6" iyz="0" izz="1e-6" />
+    </inertial>
+  </link>
+  <!-- Gazebo plugin -->
+  <gazebo reference="${tf_prefix}_camera_link2">
+    <sensor type="camera" name="camera2">
+      <update_rate>100.0</update_rate>
+      <camera name="camera2">
+        <horizontal_fov>1.3962634</horizontal_fov>
+        <image>
+          <width>800</width>
+          <height>800</height>
+          <format>R8G8B8</format>
+        </image>
+        <clip>
+          <near>0.02</near>
+          <far>300</far>
+        </clip>
+        <noise>
+          <type>gaussian</type>
+          <mean>0.0</mean>
+          <stddev>0.007</stddev>
+        </noise>
+      </camera>
+      <plugin name="camera_controller" filename="libgazebo_ros_camera.so">
+        <alwaysOn>true</alwaysOn>
+        <updateRate>100.0</updateRate>
+        <cameraName>camera2</cameraName>
+        <imageTopicName>image_raw_camera2</imageTopicName>
+        <cameraInfoTopicName>camera_info2</cameraInfoTopicName>
+        <frameName>${tf_prefix}_camera_link2</frameName>
+        <hackBaseline>0.07</hackBaseline>
+        <distortionK1>0.0</distortionK1>
+        <distortionK2>0.0</distortionK2>
+        <distortionK3>0.0</distortionK3>
+        <distortionT1>0.0</distortionT1>
+        <distortionT2>0.0</distortionT2>
       </plugin>
+    </sensor>
   </gazebo>
-  <xacro:controller_plugin_gazebo robot_namespace=""/>
 </robot>
